File: hardware/constellation/constellation.kicad_sch (KiCad schematic)
At the start: 31 parts

Commit message: Roughly placed all the LEDs
Parts:
- removed D1, D10, D11, D12, D13, D14, D15, D16, D17, D18, D19, D2, D20, D21, D22, D23, D24, D25, D26, D27, D28, D29, D3, D30, D31, D4, D5, D6, D7, D8, D9: XL-1010RGBC-WS2812B, SWS-Library:XL-1010RGBC-WS2812B, symbol __sws_jlpcb:XL-1010RGBC-WS2812B
- added TP1, TP10, TP100, TP101, TP102, TP103, TP104, TP105, TP106, TP107, TP108, TP109, TP11, TP110, TP111, TP112, TP113, TP114, TP115, TP116, TP117, TP118, TP119, TP12, TP120, TP121, TP122, TP123, TP124, TP125, TP126, TP127, TP128, TP129, TP13, TP130, TP131, TP132, TP133, TP134, TP135, TP136, TP137, TP138, TP139, TP14, TP140, TP141, TP142, TP143, TP144, TP145, TP146, TP147, TP148, TP149, TP15, TP150, TP151, TP152, TP153, TP154, TP155, TP156, TP157, TP158, TP159, TP16, TP160, TP161, TP162, TP163, TP164, TP165, TP166, TP167, TP168, TP169, TP17, TP170, TP171, TP172, TP173, TP174, TP175, TP176, TP177, TP178, TP179, TP18, TP180, TP181, TP182, TP183, TP184, TP185, TP186, TP187, TP188, TP189, TP19, TP190, TP191, TP192, TP193, TP194, TP195, TP196, TP197, TP198, TP199, TP2, TP20, TP200, TP201, TP202, TP203, TP204, TP205, TP206, TP207, TP208, TP209, TP21, TP210, TP211, TP212, TP213, TP214, TP215, TP216, TP217, TP218, TP219, TP22, TP220, TP221, TP222, TP223, TP224, TP225, TP226, TP227, TP228, TP229, TP23, TP230, TP231, TP232, TP233, TP234, TP235, TP236, TP237, TP238, TP239, TP24, TP240, TP241, TP242, TP243, TP244, TP245, TP246, TP247, TP248, TP249, TP25, TP250, TP251, TP252, TP253, TP254, TP255, TP256, TP257, TP258, TP259, TP26, TP260, TP261, TP262, TP263, TP264, TP265, TP266, TP267, TP268, TP269, TP27, TP270, TP28, TP29, TP3, TP30, TP31, TP32, TP33, TP34, TP35, TP36, TP37, TP38, TP39, TP4, TP40, TP41, TP42, TP43, TP44, TP45, TP46, TP47, TP48, TP49, TP5, TP50, TP51, TP52, TP53, TP54, TP55, TP56, TP57, TP58, TP59, TP6, TP60, TP61, TP62, TP63, TP64, TP65, TP66, TP67, TP68, TP69, TP7, TP70, TP71, TP72, TP73, TP74, TP75, TP76, TP77, TP78, TP79, TP8, TP80, TP81, TP82, TP83, TP84, TP85, TP86, TP87, TP88, TP89, TP9, TP90, TP91, TP92, TP93, TP94, TP95, TP96, TP97, TP98, TP99: TestPoint, TestPoint:TestPoint_Pad_D1.5mm, symbol Connector:TestPoint
- added U1, U10, U100, U101, U102, U103, U104, U105, U106, U107, U108, U109, U11, U110, U111, U112, U113, U114, U115, U116, U117, U118, U119, U12, U120, U121, U122, U123, U124, U125, U126, U127, U128, U129, U13, U130, U131, U132, U133, U134, U135, U136, U137, U138, U139, U14, U140, U141, U142, U143, U144, U145, U146, U147, U148, U149, U15, U150, U151, U152, U153, U154, U155, U156, U157, U158, U159, U16, U160, U161, U162, U163, U164, U165, U166, U167, U168, U169, U17, U170, U171, U172, U173, U174, U175, U176, U177, U178, U179, U18, U180, U181, U182, U183, U184, U185, U186, U187, U188, U189, U19, U190, U191, U192, U193, U194, U195, U196, U197, U198, U199, U2, U20, U200, U201, U202, U203, U204, U205, U206, U207, U208, U209, U21, U210, U211, U212, U213, U214, U215, U216, U217, U218, U219, U22, U220, U221, U222, U223, U224, U225, U226, U227, U228, U229, U23, U230, U231, U232, U233, U234, U235, U236, U237, U238, U239, U24, U240, U241, U242, U243, U244, U245, U246, U247, U248, U249, U25, U250, U251, U252, U253, U254, U255, U256, U257, U258, U259, U26, U260, U261, U262, U263, U264, U265, U266, U27, U28, U29, U3, U30, U31, U32, U33, U34, U35, U36, U37, U38, U39, U4, U40, U41, U42, U43, U44, U45, U46, U47, U48, U49, U5, U50, U51, U52, U53, U54, U55, U56, U57, U58, U59, U6, U60, U61, U62, U63, U64, U65, U66, U67, U68, U69, U7, U70, U71, U72, U73, U74, U75, U76, U77, U78, U79, U8, U80, U81, U82, U83, U84, U85, U86, U87, U88, U89, U9, U90, U91, U92, U93, U94, U95, U96, U97, U98, U99: XL-1010RGBC, easyeda2kicad:LED-SMD_4P-L1.0-W1.0-TL_XL-1010RGBC-WS2812B, symbol __easyeda2kicad:XL-1010RGBC-WS2812B
Connections:
- net +5V: now also TP18.1, U1.2 (VDD), U10.2 (VDD), U100.2 (VDD), U101.2 (VDD), U102.2 (VDD), U103.2 (VDD), U104.2 (VDD), U105.2 (VDD), U106.2 (VDD), U107.2 (VDD), U108.2 (VDD), U109.2 (VDD), U11.2 (VDD), U110.2 (VDD), U111.2 (VDD), U112.2 (VDD), U113.2 (VDD), U114.2 (VDD), U115.2 (VDD), U116.2 (VDD), U117.2 (VDD), U118.2 (VDD), U119.2 (VDD), U12.2 (VDD), U120.2 (VDD), U121.2 (VDD), U122.2 (VDD), U123.2 (VDD), U124.2 (VDD), U125.2 (VDD), U126.2 (VDD), U127.2 (VDD), U128.2 (VDD), U129.2 (VDD), U13.2 (VDD), U130.2 (VDD), U131.2 (VDD), U132.2 (VDD), U133.2 (VDD), U134.2 (VDD), U135.2 (VDD), U136.2 (VDD), U137.2 (VDD), U138.2 (VDD), U139.2 (VDD), U14.2 (VDD), U140.2 (VDD), U141.2 (VDD), U142.2 (VDD), U143.2 (VDD), U144.2 (VDD), U145.2 (VDD), U146.2 (VDD), U147.2 (VDD), U148.2 (VDD), U149.2 (VDD), U15.2 (VDD), U150.2 (VDD), U151.2 (VDD), U152.2 (VDD), U153.2 (VDD), U154.2 (VDD), U155.2 (VDD), U156.2 (VDD), U157.2 (VDD), U158.2 (VDD), U159.2 (VDD), U16.2 (VDD), U160.2 (VDD), U161.2 (VDD), U162.2 (VDD), U163.2 (VDD), U164.2 (VDD), U165.2 (VDD), U166.2 (VDD), U167.2 (VDD), U168.2 (VDD), U169.2 (VDD), U17.2 (VDD), U170.2 (VDD), U171.2 (VDD), U172.2 (VDD), U173.2 (VDD), U174.2 (VDD), U175.2 (VDD), U176.2 (VDD), U177.2 (VDD), U178.2 (VDD), U179.2 (VDD), U18.2 (VDD), U180.2 (VDD), U181.2 (VDD), U182.2 (VDD), U183.2 (VDD), U184.2 (VDD), U185.2 (VDD), U186.2 (VDD), U187.2 (VDD), U188.2 (VDD), U189.2 (VDD), U19.2 (VDD), U190.2 (VDD), U191.2 (VDD), U192.2 (VDD), U193.2 (VDD), U194.2 (VDD), U195.2 (VDD), U196.2 (VDD), U197.2 (VDD), U198.2 (VDD), U199.2 (VDD), U2.2 (VDD), U20.2 (VDD), U200.2 (VDD), U201.2 (VDD), U202.2 (VDD), U203.2 (VDD), U204.2 (VDD), U205.2 (VDD), U206.2 (VDD), U207.2 (VDD), U208.2 (VDD), U209.2 (VDD), U21.2 (VDD), U210.2 (VDD), U211.2 (VDD), U212.2 (VDD), U213.2 (VDD), U214.2 (VDD), U215.2 (VDD), U216.2 (VDD), U217.2 (VDD), U218.2 (VDD), U219.2 (VDD), U22.2 (VDD), U220.2 (VDD), U221.2 (VDD), U222.2 (VDD), U223.2 (VDD), U224.2 (VDD), U225.2 (VDD), U226.2 (VDD), U227.2 (VDD), U228.2 (VDD), U229.2 (VDD), U23.2 (VDD), U230.2 (VDD), U231.2 (VDD), U232.2 (VDD), U233.2 (VDD), U234.2 (VDD), U235.2 (VDD), U236.2 (VDD), U237.2 (VDD), U238.2 (VDD), U239.2 (VDD), U24.2 (VDD), U240.2 (VDD), U241.2 (VDD), U242.2 (VDD), U243.2 (VDD), U244.2 (VDD), U245.2 (VDD), U246.2 (VDD), U247.2 (VDD), U248.2 (VDD), U249.2 (VDD), U25.2 (VDD), U250.2 (VDD), U251.2 (VDD), U252.2 (VDD), U253.2 (VDD), U254.2 (VDD), U255.2 (VDD), U256.2 (VDD), U257.2 (VDD), U258.2 (VDD), U259.2 (VDD), U26.2 (VDD), U260.2 (VDD), U261.2 (VDD), U262.2 (VDD), U263.2 (VDD), U264.2 (VDD), U265.2 (VDD), U266.2 (VDD), U27.2 (VDD), U28.2 (VDD), U29.2 (VDD), U3.2 (VDD), U30.2 (VDD), U31.2 (VDD), U32.2 (VDD), U33.2 (VDD), U34.2 (VDD), U35.2 (VDD), U36.2 (VDD), U37.2 (VDD), U38.2 (VDD), U39.2 (VDD), U4.2 (VDD), U40.2 (VDD), U41.2 (VDD), U42.2 (VDD), U43.2 (VDD), U44.2 (VDD), U45.2 (VDD), U46.2 (VDD), U47.2 (VDD), U48.2 (VDD), U49.2 (VDD), U5.2 (VDD), U50.2 (VDD), U51.2 (VDD), U52.2 (VDD), U53.2 (VDD), U54.2 (VDD), U55.2 (VDD), U56.2 (VDD), U57.2 (VDD), U58.2 (VDD), U59.2 (VDD), U6.2 (VDD), U60.2 (VDD), U61.2 (VDD), U62.2 (VDD), U63.2 (VDD), U64.2 (VDD), U65.2 (VDD), U66.2 (VDD), U67.2 (VDD), U68.2 (VDD), U69.2 (VDD), U7.2 (VDD), U70.2 (VDD), U71.2 (VDD), U72.2 (VDD), U73.2 (VDD), U74.2 (VDD), U75.2 (VDD), U76.2 (VDD), U77.2 (VDD), U78.2 (VDD), U79.2 (VDD), U8.2 (VDD), U80.2 (VDD), U81.2 (VDD), U82.2 (VDD), U83.2 (VDD), U84.2 (VDD), U85.2 (VDD), U86.2 (VDD), U87.2 (VDD), U88.2 (VDD), U89.2 (VDD), U9.2 (VDD), U90.2 (VDD), U91.2 (VDD), U92.2 (VDD), U93.2 (VDD), U94.2 (VDD), U95.2 (VDD), U96.2 (VDD), U97.2 (VDD), U98.2 (VDD), U99.2 (VDD)
- net GND: now also TP19.1, U1.3 (GND), U10.3 (GND), U100.3 (GND), U101.3 (GND), U102.3 (GND), U103.3 (GND), U104.3 (GND), U105.3 (GND), U106.3 (GND), U107.3 (GND), U108.3 (GND), U109.3 (GND), U11.3 (GND), U110.3 (GND), U111.3 (GND), U112.3 (GND), U113.3 (GND), U114.3 (GND), U115.3 (GND), U116.3 (GND), U117.3 (GND), U118.3 (GND), U119.3 (GND), U12.3 (GND), U120.3 (GND), U121.3 (GND), U122.3 (GND), U123.3 (GND), U124.3 (GND), U125.3 (GND), U126.3 (GND), U127.3 (GND), U128.3 (GND), U129.3 (GND), U13.3 (GND), U130.3 (GND), U131.3 (GND), U132.3 (GND), U133.3 (GND), U134.3 (GND), U135.3 (GND), U136.3 (GND), U137.3 (GND), U138.3 (GND), U139.3 (GND), U14.3 (GND), U140.3 (GND), U141.3 (GND), U142.3 (GND), U143.3 (GND), U144.3 (GND), U145.3 (GND), U146.3 (GND), U147.3 (GND), U148.3 (GND), U149.3 (GND), U15.3 (GND), U150.3 (GND), U151.3 (GND), U152.3 (GND), U153.3 (GND), U154.3 (GND), U155.3 (GND), U156.3 (GND), U157.3 (GND), U158.3 (GND), U159.3 (GND), U16.3 (GND), U160.3 (GND), U161.3 (GND), U162.3 (GND), U163.3 (GND), U164.3 (GND), U165.3 (GND), U166.3 (GND), U167.3 (GND), U168.3 (GND), U169.3 (GND), U17.3 (GND), U170.3 (GND), U171.3 (GND), U172.3 (GND), U173.3 (GND), U174.3 (GND), U175.3 (GND), U176.3 (GND), U177.3 (GND), U178.3 (GND), U179.3 (GND), U18.3 (GND), U180.3 (GND), U181.3 (GND), U182.3 (GND), U183.3 (GND), U184.3 (GND), U185.3 (GND), U186.3 (GND), U187.3 (GND), U188.3 (GND), U189.3 (GND), U19.3 (GND), U190.3 (GND), U191.3 (GND), U192.3 (GND), U193.3 (GND), U194.3 (GND), U195.3 (GND), U196.3 (GND), U197.3 (GND), U198.3 (GND), U199.3 (GND), U2.3 (GND), U20.3 (GND), U200.3 (GND), U201.3 (GND), U202.3 (GND), U203.3 (GND), U204.3 (GND), U205.3 (GND), U206.3 (GND), U207.3 (GND), U208.3 (GND), U209.3 (GND), U21.3 (GND), U210.3 (GND), U211.3 (GND), U212.3 (GND), U213.3 (GND), U214.3 (GND), U215.3 (GND), U216.3 (GND), U217.3 (GND), U218.3 (GND), U219.3 (GND), U22.3 (GND), U220.3 (GND), U221.3 (GND), U222.3 (GND), U223.3 (GND), U224.3 (GND), U225.3 (GND), U226.3 (GND), U227.3 (GND), U228.3 (GND), U229.3 (GND), U23.3 (GND), U230.3 (GND), U231.3 (GND), U232.3 (GND), U233.3 (GND), U234.3 (GND), U235.3 (GND), U236.3 (GND), U237.3 (GND), U238.3 (GND), U239.3 (GND), U24.3 (GND), U240.3 (GND), U241.3 (GND), U242.3 (GND), U243.3 (GND), U244.3 (GND), U245.3 (GND), U246.3 (GND), U247.3 (GND), U248.3 (GND), U249.3 (GND), U25.3 (GND), U250.3 (GND), U251.3 (GND), U252.3 (GND), U253.3 (GND), U254.3 (GND), U255.3 (GND), U256.3 (GND), U257.3 (GND), U258.3 (GND), U259.3 (GND), U26.3 (GND), U260.3 (GND), U261.3 (GND), U262.3 (GND), U263.3 (GND), U264.3 (GND), U265.3 (GND), U266.3 (GND), U27.3 (GND), U28.3 (GND), U29.3 (GND), U3.3 (GND), U30.3 (GND), U31.3 (GND), U32.3 (GND), U33.3 (GND), U34.3 (GND), U35.3 (GND), U36.3 (GND), U37.3 (GND), U38.3 (GND), U39.3 (GND), U4.3 (GND), U40.3 (GND), U41.3 (GND), U42.3 (GND), U43.3 (GND), U44.3 (GND), U45.3 (GND), U46.3 (GND), U47.3 (GND), U48.3 (GND), U49.3 (GND), U5.3 (GND), U50.3 (GND), U51.3 (GND), U52.3 (GND), U53.3 (GND), U54.3 (GND), U55.3 (GND), U56.3 (GND), U57.3 (GND), U58.3 (GND), U59.3 (GND), U6.3 (GND), U60.3 (GND), U61.3 (GND), U62.3 (GND), U63.3 (GND), U64.3 (GND), U65.3 (GND), U66.3 (GND), U67.3 (GND), U68.3 (GND), U69.3 (GND), U7.3 (GND), U70.3 (GND), U71.3 (GND), U72.3 (GND), U73.3 (GND), U74.3 (GND), U75.3 (GND), U76.3 (GND), U77.3 (GND), U78.3 (GND), U79.3 (GND), U8.3 (GND), U80.3 (GND), U81.3 (GND), U82.3 (GND), U83.3 (GND), U84.3 (GND), U85.3 (GND), U86.3 (GND), U87.3 (GND), U88.3 (GND), U89.3 (GND), U9.3 (GND), U90.3 (GND), U91.3 (GND), U92.3 (GND), U93.3 (GND), U94.3 (GND), U95.3 (GND), U96.3 (GND), U97.3 (GND), U98.3 (GND), U99.3 (GND)
- new net: TP75.1, U71.1 (DOUT), U72.4 (DIN)
- new net: TP262.1, U258.1 (DOUT), U259.4 (DIN)
- new net: TP261.1, U257.1 (DOUT), U258.4 (DIN)
- new net: TP242.1, U238.1 (DOUT), U239.4 (DIN)
- new net: TP241.1, U237.1 (DOUT), U238.4 (DIN)
- new net: TP147.1, U143.1 (DOUT), U144.4 (DIN)
- new net: TP47.1, U43.1 (DOUT), U44.4 (DIN)
- new net: TP248.1, U244.1 (DOUT), U245.4 (DIN)
- new net: TP256.1, U252.1 (DOUT), U253.4 (DIN)
- new net: TP255.1, U251.1 (DOUT), U252.4 (DIN)
- new net: TP182.1, U178.1 (DOUT), U179.4 (DIN)
- new net: TP163.1, U159.1 (DOUT), U160.4 (DIN)
- new net: TP63.1, U59.1 (DOUT), U60.4 (DIN)
- new net: TP2.1, U2.1 (DOUT), U3.4 (DIN)
- new net: TP1.1, U1.1 (DOUT), U2.4 (DIN)
- new net: TP139.1, U135.1 (DOUT), U136.4 (DIN)
- new net: TP206.1, U202.1 (DOUT), U203.4 (DIN)
- new net: TP205.1, U201.1 (DOUT), U202.4 (DIN)
- new net: TP100.1, U96.1 (DOUT), U97.4 (DIN)
- new net: TP69.1, U65.1 (DOUT), U66.4 (DIN)
- new net: TP128.1, U124.1 (DOUT), U125.4 (DIN)
- new net: TP127.1, U123.1 (DOUT), U124.4 (DIN)
- new net: TP260.1, U256.1 (DOUT), U257.4 (DIN)
- new net: TP232.1, U228.1 (DOUT), U229.4 (DIN)
- new net: TP231.1, U227.1 (DOUT), U228.4 (DIN)
- new net: TP235.1, U231.1 (DOUT), U232.4 (DIN)
- new net: TP234.1, U230.1 (DOUT), U231.4 (DIN)
- new net: TP233.1, U229.1 (DOUT), U230.4 (DIN)
- new net: TP193.1, U189.1 (DOUT), U190.4 (DIN)
- new net: TP237.1, U233.1 (DOUT), U234.4 (DIN)
- new net: TP236.1, U232.1 (DOUT), U233.4 (DIN)
- new net: TP194.1, U190.1 (DOUT), U191.4 (DIN)
- new net: TP149.1, U145.1 (DOUT), U146.4 (DIN)
- new net: TP189.1, U185.1 (DOUT), U186.4 (DIN)
- new net: TP72.1, U68.1 (DOUT), U69.4 (DIN)
- new net: TP125.1, U121.1 (DOUT), U122.4 (DIN)
- new net: TP124.1, U120.1 (DOUT), U121.4 (DIN)
- new net: TP11.1, U11.1 (DOUT), U12.4 (DIN)
- new net: TP179.1, U175.1 (DOUT), U176.4 (DIN)
- new net: TP38.1, U34.1 (DOUT), U35.4 (DIN)
- new net: TP216.1, U212.1 (DOUT), U213.4 (DIN)
- new net: TP215.1, U211.1 (DOUT), U212.4 (DIN)
- new net: TP176.1, U172.1 (DOUT), U173.4 (DIN)
- new net: TP175.1, U171.1 (DOUT), U172.4 (DIN)
- new net: TP4.1, U4.1 (DOUT), U5.4 (DIN)
- new net: TP268.1, U264.1 (DOUT), U265.4 (DIN)
- new net: TP196.1, U192.1 (DOUT), U193.4 (DIN)
- new net: TP195.1, U191.1 (DOUT), U192.4 (DIN)
- new net: TP27.1, U23.1 (DOUT), U24.4 (DIN)
- new net: TP92.1, U88.1 (DOUT), U89.4 (DIN)
- new net: TP3.1, U3.1 (DOUT), U4.4 (DIN)
- new net: TP7.1, U7.1 (DOUT), U8.4 (DIN)
- new net: TP6.1, U6.1 (DOUT), U7.4 (DIN)
- new net: TP118.1, U114.1 (DOUT), U115.4 (DIN)
- new net: TP49.1, U45.1 (DOUT), U46.4 (DIN)
- new net: TP46.1, U42.1 (DOUT), U43.4 (DIN)
- new net: TP45.1, U41.1 (DOUT), U42.4 (DIN)
- new net: TP67.1, U63.1 (DOUT), U64.4 (DIN)
- new net: TP66.1, U62.1 (DOUT), U63.4 (DIN)
- new net: TP115.1, U111.1 (DOUT), U112.4 (DIN)
- new net: TP114.1, U110.1 (DOUT), U111.4 (DIN)
- new net: TP30.1, U26.1 (DOUT), U27.4 (DIN)
- new net: TP117.1, U113.1 (DOUT), U114.4 (DIN)
- new net: TP107.1, U103.1 (DOUT), U104.4 (DIN)
- new net: TP106.1, U102.1 (DOUT), U103.4 (DIN)
- new net: TP213.1, U209.1 (DOUT), U210.4 (DIN)
- new net: TP212.1, U208.1 (DOUT), U209.4 (DIN)
- new net: TP126.1, U122.1 (DOUT), U123.4 (DIN)
- new net: TP52.1, U48.1 (DOUT), U49.4 (DIN)
- new net: TP51.1, U47.1 (DOUT), U48.4 (DIN)
- new net: TP8.1, U8.1 (DOUT), U9.4 (DIN)
- new net: TP150.1, U146.1 (DOUT), U147.4 (DIN)
- new net: TP116.1, U112.1 (DOUT), U113.4 (DIN)
- new net: TP166.1, U162.1 (DOUT), U163.4 (DIN)
- new net: TP225.1, U221.1 (DOUT), U222.4 (DIN)
- new net: TP224.1, U220.1 (DOUT), U221.4 (DIN)
- new net: TP36.1, U32.1 (DOUT), U33.4 (DIN)
- new net: TP177.1, U173.1 (DOUT), U174.4 (DIN)
- new net: TP23.1, U19.1 (DOUT), U20.4 (DIN)
- new net: TP64.1, U60.1 (DOUT), U61.4 (DIN)
- new net: TP227.1, U223.1 (DOUT), U224.4 (DIN)
- new net: TP238.1, U234.1 (DOUT), U235.4 (DIN)
- new net: TP12.1, U12.1 (DOUT), U13.4 (DIN)
- new net: TP37.1, U33.1 (DOUT), U34.4 (DIN)
- new net: TP145.1, U141.1 (DOUT), U142.4 (DIN)
- new net: TP144.1, U140.1 (DOUT), U141.4 (DIN)
- new net: TP181.1, U177.1 (DOUT), U178.4 (DIN)
- new net: TP5.1, U5.1 (DOUT), U6.4 (DIN)
- new net: TP158.1, U154.1 (DOUT), U155.4 (DIN)
- new net: TP83.1, U79.1 (DOUT), U80.4 (DIN)
- new net: TP82.1, U78.1 (DOUT), U79.4 (DIN)
- new net: TP186.1, U182.1 (DOUT), U183.4 (DIN)
- new net: TP162.1, U158.1 (DOUT), U159.4 (DIN)
- new net: TP263.1, U259.1 (DOUT), U260.4 (DIN)
- new net: TP259.1, U255.1 (DOUT), U256.4 (DIN)
- new net: TP129.1, U125.1 (DOUT), U126.4 (DIN)
- new net: TP94.1, U90.1 (DOUT), U91.4 (DIN)
- new net: TP93.1, U89.1 (DOUT), U90.4 (DIN)
- new net: TP172.1, U168.1 (DOUT), U169.4 (DIN)
- new net: TP171.1, U167.1 (DOUT), U168.4 (DIN)
- new net: TP71.1, U67.1 (DOUT), U68.4 (DIN)
- new net: TP121.1, U117.1 (DOUT), U118.4 (DIN)
- new net: TP252.1, U248.1 (DOUT), U249.4 (DIN)
- new net: TP251.1, U247.1 (DOUT), U248.4 (DIN)
- new net: TP185.1, U181.1 (DOUT), U182.4 (DIN)
- new net: TP184.1, U180.1 (DOUT), U181.4 (DIN)
- new net: TP55.1, U51.1 (DOUT), U52.4 (DIN)
- new net: TP110.1, U106.1 (DOUT), U107.4 (DIN)
- new net: TP109.1, U105.1 (DOUT), U106.4 (DIN)
- new net: TP267.1, U263.1 (DOUT), U264.4 (DIN)
- new net: TP266.1, U262.1 (DOUT), U263.4 (DIN)
- new net: TP54.1, U50.1 (DOUT), U51.4 (DIN)
- new net: TP53.1, U49.1 (DOUT), U50.4 (DIN)
- new net: TP228.1, U224.1 (DOUT), U225.4 (DIN)
- new net: TP91.1, U87.1 (DOUT), U88.4 (DIN)
- new net: TP15.1, U15.1 (DOUT), U16.4 (DIN)
- new net: TP102.1, U98.1 (DOUT), U99.4 (DIN)
- new net: TP101.1, U97.1 (DOUT), U98.4 (DIN)
- new net: TP24.1, U20.1 (DOUT), U21.4 (DIN)
- new net: TP264.1, U260.1 (DOUT), U261.4 (DIN)
- new net: TP191.1, U187.1 (DOUT), U188.4 (DIN)
- new net: TP190.1, U186.1 (DOUT), U187.4 (DIN)
- new net: TP25.1, U21.1 (DOUT), U22.4 (DIN)
- new net: TP202.1, U198.1 (DOUT), U199.4 (DIN)
- new net: TP10.1, U10.1 (DOUT), U11.4 (DIN)
- new net: TP9.1, U10.4 (DIN), U9.1 (DOUT)
- new net: TP48.1, U44.1 (DOUT), U45.4 (DIN)
- new net: TP167.1, U163.1 (DOUT), U164.4 (DIN)
- new net: TP98.1, U94.1 (DOUT), U95.4 (DIN)
- new net: TP97.1, U93.1 (DOUT), U94.4 (DIN)
- new net: TP58.1, U54.1 (DOUT), U55.4 (DIN)
- new net: TP123.1, U119.1 (DOUT), U120.4 (DIN)
- new net: TP140.1, U136.1 (DOUT), U137.4 (DIN)
- new net: TP96.1, U92.1 (DOUT), U93.4 (DIN)
- new net: TP95.1, U91.1 (DOUT), U92.4 (DIN)
- new net: TP137.1, U133.1 (DOUT), U134.4 (DIN)
- new net: TP136.1, U132.1 (DOUT), U133.4 (DIN)
- new net: TP219.1, U215.1 (DOUT), U216.4 (DIN)
- new net: TP269.1, U265.1 (DOUT), U266.4 (DIN)
- new net: TP207.1, U203.1 (DOUT), U204.4 (DIN)
- new net: TP84.1, U80.1 (DOUT), U81.4 (DIN)
- new net: TP87.1, U83.1 (DOUT), U84.4 (DIN)
- new net: TP230.1, U226.1 (DOUT), U227.4 (DIN)
- new net: TP113.1, U109.1 (DOUT), U110.4 (DIN)
- new net: TP86.1, U82.1 (DOUT), U83.4 (DIN)
- new net: TP85.1, U81.1 (DOUT), U82.4 (DIN)
- new net: TP80.1, U76.1 (DOUT), U77.4 (DIN)
- new net: TP119.1, U115.1 (DOUT), U116.4 (DIN)
- new net: TP154.1, U150.1 (DOUT), U151.4 (DIN)
- new net: TP153.1, U149.1 (DOUT), U150.4 (DIN)
- new net: TP22.1, U18.1 (DOUT), U19.4 (DIN)
- new net: TP79.1, U75.1 (DOUT), U76.4 (DIN)
- new net: TP78.1, U74.1 (DOUT), U75.4 (DIN)
- new net: TP62.1, U58.1 (DOUT), U59.4 (DIN)
- new net: TP180.1, U176.1 (DOUT), U177.4 (DIN)
- new net: TP56.1, U52.1 (DOUT), U53.4 (DIN)
- new net: TP111.1, U107.1 (DOUT), U108.4 (DIN)
- new net: TP31.1, U27.1 (DOUT), U28.4 (DIN)
- new net: TP217.1, U213.1 (DOUT), U214.4 (DIN)
- new net: TP151.1, U147.1 (DOUT), U148.4 (DIN)
- new net: TP239.1, U235.1 (DOUT), U236.4 (DIN)
- new net: TP42.1, U38.1 (DOUT), U39.4 (DIN)
- new net: TP165.1, U161.1 (DOUT), U162.4 (DIN)
- new net: TP164.1, U160.1 (DOUT), U161.4 (DIN)
- new net: TP103.1, U100.4 (DIN), U99.1 (DOUT)
- new net: TP168.1, U164.1 (DOUT), U165.4 (DIN)
- new net: TP74.1, U70.1 (DOUT), U71.4 (DIN)
- new net: TP108.1, U104.1 (DOUT), U105.4 (DIN)
- new net: TP223.1, U219.1 (DOUT), U220.4 (DIN)
- new net: TP112.1, U108.1 (DOUT), U109.4 (DIN)
- new net: TP204.1, U200.1 (DOUT), U201.4 (DIN)
- new net: TP203.1, U199.1 (DOUT), U200.4 (DIN)
- new net: TP16.1, U16.1 (DOUT), U17.4 (DIN)
- new net: TP132.1, U128.1 (DOUT), U129.4 (DIN)
- new net: TP200.1, U196.1 (DOUT), U197.4 (DIN)
- new net: TP199.1, U195.1 (DOUT), U196.4 (DIN)
- new net: TP209.1, U205.1 (DOUT), U206.4 (DIN)
- new net: TP221.1, U217.1 (DOUT), U218.4 (DIN)
- new net: TP220.1, U216.1 (DOUT), U217.4 (DIN)
- new net: TP60.1, U56.1 (DOUT), U57.4 (DIN)
- new net: TP183.1, U179.1 (DOUT), U180.4 (DIN)
- new net: TP26.1, U22.1 (DOUT), U23.4 (DIN)
- new net: TP41.1, U37.1 (DOUT), U38.4 (DIN)
- new net: TP249.1, U245.1 (DOUT), U246.4 (DIN)
- new net: TP240.1, U236.1 (DOUT), U237.4 (DIN)
- new net: TP229.1, U225.1 (DOUT), U226.4 (DIN)
- new net: TP245.1, U241.1 (DOUT), U242.4 (DIN)
- new net: TP244.1, U240.1 (DOUT), U241.4 (DIN)
- new net: TP29.1, U25.1 (DOUT), U26.4 (DIN)
- new net: TP28.1, U24.1 (DOUT), U25.4 (DIN)
- new net: TP148.1, U144.1 (DOUT), U145.4 (DIN)
- new net: TP211.1, U207.1 (DOUT), U208.4 (DIN)
- new net: TP141.1, U137.1 (DOUT), U138.4 (DIN)
- new net: TP188.1, U184.1 (DOUT), U185.4 (DIN)
- new net: TP246.1, U242.1 (DOUT), U243.4 (DIN)
- new net: TP34.1, U30.1 (DOUT), U31.4 (DIN)
- new net: TP40.1, U36.1 (DOUT), U37.4 (DIN)
- new net: TP39.1, U35.1 (DOUT), U36.4 (DIN)
- new net: TP130.1, U126.1 (DOUT), U127.4 (DIN)
- new net: TP57.1, U53.1 (DOUT), U54.4 (DIN)
- new net: TP214.1, U210.1 (DOUT), U211.4 (DIN)
- new net: TP43.1, U39.1 (DOUT), U40.4 (DIN)
- new net: TP138.1, U134.1 (DOUT), U135.4 (DIN)
- new net: TP169.1, U165.1 (DOUT), U166.4 (DIN)
- new net: TP152.1, U148.1 (DOUT), U149.4 (DIN)
- new net: TP254.1, U250.1 (DOUT), U251.4 (DIN)
- new net: TP253.1, U249.1 (DOUT), U250.4 (DIN)
- new net: TP14.1, U14.1 (DOUT), U15.4 (DIN)
- new net: TP187.1, U183.1 (DOUT), U184.4 (DIN)
- new net: TP155.1, U151.1 (DOUT), U152.4 (DIN)
- new net: TP90.1, U86.1 (DOUT), U87.4 (DIN)
- new net: TP222.1, U218.1 (DOUT), U219.4 (DIN)
- new net: TP68.1, U64.1 (DOUT), U65.4 (DIN)
- new net: TP161.1, U157.1 (DOUT), U158.4 (DIN)
- new net: TP122.1, U118.1 (DOUT), U119.4 (DIN)
- new net: TP218.1, U214.1 (DOUT), U215.4 (DIN)
- new net: TP173.1, U169.1 (DOUT), U170.4 (DIN)
- new net: TP32.1, U28.1 (DOUT), U29.4 (DIN)
- new net: TP198.1, U194.1 (DOUT), U195.4 (DIN)
- new net: TP81.1, U77.1 (DOUT), U78.4 (DIN)
- new net: TP257.1, U253.1 (DOUT), U254.4 (DIN)
- new net: TP208.1, U204.1 (DOUT), U205.4 (DIN)
- new net: TP156.1, U152.1 (DOUT), U153.4 (DIN)
- new net: TP61.1, U57.1 (DOUT), U58.4 (DIN)
- new net: TP146.1, U142.1 (DOUT), U143.4 (DIN)
- new net: TP135.1, U131.1 (DOUT), U132.4 (DIN)
- new net: TP134.1, U130.1 (DOUT), U131.4 (DIN)
- new net: TP89.1, U85.1 (DOUT), U86.4 (DIN)
- new net: TP258.1, U254.1 (DOUT), U255.4 (DIN)
- new net: TP157.1, U153.1 (DOUT), U154.4 (DIN)
- new net: TP35.1, U31.1 (DOUT), U32.4 (DIN)
- new net: TP160.1, U156.1 (DOUT), U157.4 (DIN)
- new net: TP50.1, U46.1 (DOUT), U47.4 (DIN)
- new net: TP131.1, U127.1 (DOUT), U128.4 (DIN)
- new net: TP13.1, U13.1 (DOUT), U14.4 (DIN)
- new net: TP170.1, U166.1 (DOUT), U167.4 (DIN)
- new net: TP77.1, U73.1 (DOUT), U74.4 (DIN)
- new net: TP142.1, U138.1 (DOUT), U139.4 (DIN)
- new net: TP247.1, U243.1 (DOUT), U244.4 (DIN)
- new net: TP65.1, U61.1 (DOUT), U62.4 (DIN)
- new net: TP105.1, U101.1 (DOUT), U102.4 (DIN)
- new net: TP99.1, U95.1 (DOUT), U96.4 (DIN)
- new net: TP133.1, U129.1 (DOUT), U130.4 (DIN)
- new net: TP174.1, U170.1 (DOUT), U171.4 (DIN)
- new net: TP73.1, U69.1 (DOUT), U70.4 (DIN)
- new net: TP192.1, U188.1 (DOUT), U189.4 (DIN)
- new net: TP201.1, U197.1 (DOUT), U198.4 (DIN)
- new net LED_Andromeda: TP20.1, U1.4 (DIN)
- new net LED_Aquarius: TP17.1, U17.1 (DOUT), U18.4 (DIN)
- new net LED_Aries: TP33.1, U29.1 (DOUT), U30.4 (DIN)
- new net LED_Capricornus: TP76.1, U72.1 (DOUT), U73.4 (DIN)
- new net LED_Cassiopeia: TP70.1, U66.1 (DOUT), U67.4 (DIN)
- new net LED_Cepheus: TP59.1, U55.1 (DOUT), U56.4 (DIN)
- new net LED_Cetus: TP44.1, U40.1 (DOUT), U41.4 (DIN)
- new net LED_Draco: TP88.1, U84.1 (DOUT), U85.4 (DIN)
- new net LED_Gemini: TP104.1, U100.1 (DOUT), U101.4 (DIN)
- new net LED_Hercules: TP120.1, U116.1 (DOUT), U117.4 (DIN)
- new net LED_Leo: TP143.1, U139.1 (DOUT), U140.4 (DIN)
- new net LED_OUT: TP21.1, TP270.1, U266.1 (DOUT)
- new net LED_Orion: TP159.1, U155.1 (DOUT), U156.4 (DIN)
- new net LED_Perseus: TP226.1, U222.1 (DOUT), U223.4 (DIN)
- new net LED_Pisces: TP210.1, U206.1 (DOUT), U207.4 (DIN)
- new net LED_Serpens: TP197.1, U193.1 (DOUT), U194.4 (DIN)
- new net LED_Ursa_major: TP178.1, U174.1 (DOUT), U175.4 (DIN)
- new net LED_Ursa_minor: TP243.1, U239.1 (DOUT), U240.4 (DIN)
- new net LED_Virgo: TP250.1, U246.1 (DOUT), U247.4 (DIN)
- new net LED_Vulpecula: TP265.1, U261.1 (DOUT), U262.4 (DIN)

Commit message: WIP: Connecting paths in constellations PCB
Parts:
- removed TP1, TP10, TP100, TP101, TP102, TP103, TP104, TP105, TP106, TP107, TP108, TP109, TP11, TP110, TP111, TP112, TP113, TP114, TP115, TP116, TP117, TP118, TP119, TP12, TP120, TP121, TP122, TP123, TP124, TP125, TP126, TP127, TP128, TP129, TP13, TP130, TP131, TP132, TP133, TP134, TP135, TP136, TP137, TP138, TP139, TP14, TP140, TP141, TP142, TP143, TP144, TP145, TP146, TP147, TP148, TP149, TP15, TP150, TP151, TP152, TP153, TP154, TP155, TP156, TP157, TP158, TP159, TP16, TP160, TP161, TP162, TP163, TP164, TP165, TP166, TP167, TP168, TP169, TP17, TP170, TP171, TP172, TP173, TP174, TP175, TP176, TP177, TP178, TP179, TP18, TP180, TP181, TP182, TP183, TP184, TP185, TP186, TP187, TP188, TP189, TP19, TP190, TP191, TP192, TP193, TP194, TP195, TP196, TP197, TP198, TP199, TP2, TP20, TP200, TP201, TP202, TP203, TP204, TP205, TP206, TP207, TP208, TP209, TP21, TP210, TP211, TP212, TP213, TP214, TP215, TP216, TP217, TP218, TP219, TP22, TP220, TP221, TP222, TP223, TP224, TP225, TP226, TP227, TP228, TP229, TP23, TP230, TP231, TP232, TP233, TP234, TP235, TP236, TP237, TP238, TP239, TP24, TP240, TP241, TP242, TP243, TP244, TP245, TP246, TP247, TP248, TP249, TP25, TP250, TP251, TP252, TP253, TP254, TP255, TP256, TP257, TP258, TP259, TP26, TP260, TP261, TP262, TP263, TP264, TP265, TP266, TP267, TP268, TP269, TP27, TP270, TP28, TP29, TP3, TP30, TP31, TP32, TP33, TP34, TP35, TP36, TP37, TP38, TP39, TP4, TP40, TP41, TP42, TP43, TP44, TP45, TP46, TP47, TP48, TP49, TP5, TP50, TP51, TP52, TP53, TP54, TP55, TP56, TP57, TP58, TP59, TP6, TP60, TP61, TP62, TP63, TP64, TP65, TP66, TP67, TP68, TP69, TP7, TP70, TP71, TP72, TP73, TP74, TP75, TP76, TP77, TP78, TP79, TP8, TP80, TP81, TP82, TP83, TP84, TP85, TP86, TP87, TP88, TP89, TP9, TP90, TP91, TP92, TP93, TP94, TP95, TP96, TP97, TP98, TP99: TestPoint, TestPoint:TestPoint_Pad_D1.5mm, symbol Connector:TestPoint
- added J1, J10, J11, J12, J13, J14, J15, J16, J17, J18, J19, J22, J23, J3, J4, J5, J6, J7, J8, J9: Conn_01x04, Connector_PinHeader_2.54mm:PinHeader_1x04_P2.54mm_Vertical, symbol Connector_Generic:Conn_01x04
- added J2, J20, J21, J24, J25, J26, J27, J28, J29, J30, J31, J32, J33, J34, J35, J36, J37, J38, J39: ~, SWS-Library:constellation-edge-connector_HOLES, symbol __sws_jlpcb:constellation-edge-connector_HOLE
Connections:
- net +5V: now also J1.2 (Pin_2), J10.1 (Pin_1), J11.1 (Pin_1), J12.1 (Pin_1), J13.1 (Pin_1), J14.1 (Pin_1), J16.1 (Pin_1), J17.1 (Pin_1), J18.1 (Pin_1), J19.1 (Pin_1), J22.1 (Pin_1), J23.1 (Pin_1), J3.1 (Pin_1), J4.1 (Pin_1), J5.1 (Pin_1), J6.1 (Pin_1), J7.1 (Pin_1), J8.1 (Pin_1), J9.1 (Pin_1)
- net GND: now also J1.4 (Pin_4), J10.4 (Pin_4), J11.4 (Pin_4), J12.4 (Pin_4), J13.4 (Pin_4), J14.4 (Pin_4), J16.4 (Pin_4), J17.4 (Pin_4), J18.4 (Pin_4), J19.4 (Pin_4), J2.1 (GND), J20.1 (GND), J21.1 (GND), J22.4 (Pin_4), J23.4 (Pin_4), J24.1 (GND), J25.1 (GND), J26.1 (GND), J27.1 (GND), J28.1 (GND), J29.1 (GND), J3.4 (Pin_4), J30.1 (GND), J31.1 (GND), J32.1 (GND), J33.1 (GND), J34.1 (GND), J35.1 (GND), J36.1 (GND), J37.1 (GND), J38.1 (GND), J39.1 (GND), J4.4 (Pin_4), J5.4 (Pin_4), J6.4 (Pin_4), J7.4 (Pin_4), J8.4 (Pin_4), J9.4 (Pin_4)
- net LED_Andromeda: now also J1.3 (Pin_3), J3.2 (Pin_2)
- net LED_Aquarius: now also J3.3 (Pin_3), J4.2 (Pin_2)
- net LED_Aries: now also J4.3 (Pin_3), J5.2 (Pin_2)
- net LED_Capricornus: now also J8.3 (Pin_3), J9.2 (Pin_2)
- net LED_Cassiopeia: now also J7.3 (Pin_3), J8.2 (Pin_2)
- net LED_Cepheus: now also J6.3 (Pin_3), J7.2 (Pin_2)
- net LED_Cetus: now also J5.3 (Pin_3), J6.2 (Pin_2)
- net LED_Draco: now also J10.2 (Pin_2), J9.3 (Pin_3)
- net LED_Gemini: now also J10.3 (Pin_3), J11.2 (Pin_2)
- net LED_Hercules: now also J11.3 (Pin_3), J12.2 (Pin_2)
- net LED_Leo: now also J12.3 (Pin_3), J13.2 (Pin_2)
- net LED_OUT: now also J1.1 (Pin_1), J23.3 (Pin_3)
- net LED_Orion: now also J13.3 (Pin_3), J14.2 (Pin_2)
- net LED_Perseus: now also J17.3 (Pin_3), J18.2 (Pin_2)
- net LED_Pisces: now also J16.3 (Pin_3), J17.2 (Pin_2)
- net LED_Serpens: now also J16.2 (Pin_2)
- net LED_Ursa_major: now also J14.3 (Pin_3)
- net LED_Ursa_minor: now also J18.3 (Pin_3), J19.2 (Pin_2)
- net LED_Virgo: now also J19.3 (Pin_3), J22.2 (Pin_2)
- net LED_Vulpecula: now also J22.3 (Pin_3), J23.2 (Pin_2)

Commit message: Finished DRC
Connections:
- net +5V: now also J15.1 (Pin_1)
- net GND: now also J15.4 (Pin_4)
- net LED_Serpens: now also J15.3 (Pin_3)
- net LED_Ursa_major: now also J15.2 (Pin_2)
Other:
- moved on the sheet: J15
Changed lines of the file:
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@@
 	(global_label "LED_Ursa_major"
 		(shape output)
-		(at 109.2525 427.9406 0)
+		(at 107.95 427.99 0)
 		(fields_autoplaced yes)
 		(effects
@@
 		)
 		(property "Intersheetrefs" "${INTERSHEET_REFS}"
-			(at 127.2961 427.9406 0)
+			(at 125.9936 427.99 0)
 			(effects
 				(font
@@
 	(global_label "LED_Serpens"
 		(shape input)
-		(at 109.2525 425.4006 0)
+		(at 107.95 425.45 0)
 		(fields_autoplaced yes)
 		(effects
@@
 		)
 		(property "Intersheetrefs" "${INTERSHEET_REFS}"
-			(at 124.1514 425.4006 0)
+			(at 122.8489 425.45 0)
 			(effects
 				(font
@@
 	(symbol
 		(lib_id "power:+5V")
-		(at 109.2525 430.4806 270)
+		(at 107.95 430.53 270)
 		(unit 1)
 		(exclude_from_sim no)
@@
 		(dnp no)
 		(property "Reference" "#PWR066"
-			(at 105.4425 430.4806 0)
+			(at 104.14 430.53 0)
 			(effects
 				(font
@@
 		)
 		(property "Value" "+5V"
-			(at 111.5385 430.4806 90)
+			(at 110.236 430.53 90)
 			(effects
 				(font
@@
 		)
 		(property "Footprint" ""
-			(at 109.2525 430.4806 0)
+			(at 107.95 430.53 0)
 			(effects
 				(font
@@
 		)
 		(property "Datasheet" ""
-			(at 109.2525 430.4806 0)
+			(at 107.95 430.53 0)
 			(effects
 				(font
@@
 		)
 		(property "Description" "Power symbol creates a global label with name \"+5V\""
-			(at 109.2525 430.4806 0)
+			(at 107.95 430.53 0)
 			(effects
 				(font
@@
 	(symbol
 		(lib_id "Connector_Generic:Conn_01x04")
-		(at 104.14 427.99 180)
+		(at 102.87 427.99 180)
 		(unit 1)
 		(exclude_from_sim no)
@@
 		(fields_autoplaced yes)
 		(property "Reference" "J15"
-			(at 104.14 416.56 0)
+			(at 102.87 416.56 0)
 			(effects
 				(font
@@
 		)
 		(property "Value" "Conn_01x04"
-			(at 104.14 419.1 0)
+			(at 102.87 419.1 0)
 			(effects
 				(font
@@
 		)
 		(property "Footprint" "Connector_PinHeader_2.54mm:PinHeader_1x04_P2.54mm_Vertical"
-			(at 104.14 427.99 0)
+			(at 102.87 427.99 0)
 			(effects
 				(font
@@
 		)
 		(property "Datasheet" "~"
-			(at 104.14 427.99 0)
+			(at 102.87 427.99 0)
 			(effects
 				(font
@@
 		)
 		(property "Description" "Generic connector, single row, 01x04, script generated (kicad-library-utils/schlib/autogen/connector/)"
-			(at 104.14 427.99 0)
+			(at 102.87 427.99 0)
 			(effects
 				(font
@@
 	(symbol
 		(lib_id "power:GND")
-		(at 109.2525 422.8606 90)
+		(at 107.95 422.91 90)
 		(unit 1)
 		(exclude_from_sim no)
@@
 		(dnp no)
 		(property "Reference" "#PWR065"
-			(at 115.6025 422.8606 0)
+			(at 114.3 422.91 0)
 			(effects
 				(font
@@
 		)
 		(property "Value" "GND"
-			(at 111.5385 422.8606 90)
+			(at 110.236 422.91 90)
 			(effects
 				(font
@@
 		)
 		(property "Footprint" ""
-			(at 109.2525 422.8606 0)
+			(at 107.95 422.91 0)
 			(effects
 				(font
@@
 		)
 		(property "Datasheet" ""
-			(at 109.2525 422.8606 0)
+			(at 107.95 422.91 0)
 			(effects
 				(font
@@
 		)
 		(property "Description" "Power symbol creates a global label with name \"GND\" , ground"
-			(at 109.2525 422.8606 0)
+			(at 107.95 422.91 0)
 			(effects
 				(font

Commit message: Final touches and updated readme
Parts:
- added C1, C10, C11, C12, C13, C14, C15, C16, C17, C18, C19, C2, C20, C21, C22, C23, C24, C25, C26, C27, C28, C29, C3, C30, C31, C32, C33, C34, C35, C36, C37, C38, C4, C5, C6, C7, C8, C9: 10V 10uF, Capacitor_SMD:C_0603_1608Metric, symbol Device:C
- added R1: R0, Resistor_SMD:R_0402_1005Metric, symbol __sws_jlpcb:R0
- J1, J10, J11, J12, J13, J14, J15, J16, J17, J18, J19, J22, J23, J3, J4, J5, J6, J7, J8, J9: now not fitted
Connections:
- net +5V: now also C1.2, C10.2, C11.2, C12.2, C13.2, C14.2, C15.2, C16.2, C17.2, C18.2, C19.2, C2.2, C20.2, C21.2, C22.2, C23.2, C24.2, C25.2, C26.2, C27.2, C28.2, C29.2, C3.2, C30.2, C31.2, C32.2, C33.2, C34.2, C35.2, C36.2, C37.2, C38.2, C4.2, C5.2, C6.2, C7.2, C8.2, C9.2, R1.1, R1.2
- net GND: now also C1.1, C10.1, C11.1, C12.1, C13.1, C14.1, C15.1, C16.1, C17.1, C18.1, C19.1, C2.1, C20.1, C21.1, C22.1, C23.1, C24.1, C25.1, C26.1, C27.1, C28.1, C29.1, C3.1, C30.1, C31.1, C32.1, C33.1, C34.1, C35.1, C36.1, C37.1, C38.1, C4.1, C5.1, C6.1, C7.1, C8.1, C9.1

Commit message: Added Xiao RP2040 footprint
Parts:
- added J40, J41: Conn_01x07, Connector_PinHeader_2.54mm:PinHeader_1x07_P2.54mm_Vertical, symbol Connector_Generic:Conn_01x07
- added U267: MOUDLE-SEEEDUINO-XIAO, XIAO RP2040:MOUDLE14P-SMD-2.54-21X17.8MM, symbol XIAO RP2040:MOUDLE-SEEEDUINO-XIAO
Connections:
- net +5V: now also J41.1 (Pin_1), U267.14 (5V)
- net GND: now also J41.2 (Pin_2), U267.13 (GND)
- net LED_Andromeda: now also J40.7 (Pin_7), U267.1 (PA02_A0_D0)
- new net: J41.3 (Pin_3), U267.12 (3V3)
- new net: J41.4 (Pin_4), U267.11 (PA6_A10_D10_MOSI)
- new net: J41.5 (Pin_5), U267.10 (PA5_A9_D9_MISO)
- new net: J41.6 (Pin_6), U267.9 (PA7_A8_D8_SCK)
- new net: J41.7 (Pin_7), U267.8 (PB09_A7_D7_RX)
- new net: J40.1 (Pin_1), U267.7 (PB08_A6_D6_TX)
- new net: J40.2 (Pin_2), U267.6 (PA9_A5_D5_SCL)
- new net: J40.3 (Pin_3), U267.5 (PA8_A4_D4_SDA)
- new net: J40.4 (Pin_4), U267.4 (PA11_A3_D3)
- new net: J40.5 (Pin_5), U267.3 (PA10_A2_D2)
- new net: J40.6 (Pin_6), U267.2 (PA4_A1_D1)
Other:
- moved on the sheet: C1, C10, C11, C12, C13, C14, C15, C16, C17, C18, C19, C2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
